Commit message: add a bin-picking environment, and an environment with objects

File: panda_four_description/urdf/panda_four_binpick.urdf (robot description, URDF)
Before this commit: robot panda, 56 links, 55 joints
Links:
- removed link crate
- removed link crate0
- removed link crate1
- removed link crate2
- removed link lamp0
- removed link lamp1
- removed link lamp2
- added link box1_bottom_plate; collision box size=0.5 0.5 0.02; visual box size=0.5 0.5 0.02
- added link box1_bottom_plate_back; collision box size=0.5 0.02 0.5; visual box size=0.5 0.02 0.5
- added link box1_bottom_plate_front; collision box size=0.5 0.02 0.5; visual box size=0.5 0.02 0.5
- added link box1_bottom_plate_left; collision box size=0.02 0.5 0.5; visual box size=0.02 0.5 0.5
- added link box1_bottom_plate_right; collision box size=0.02 0.5 0.5; visual box size=0.02 0.5 0.5
- added link box2_bottom_plate; collision box size=0.5 0.5 0.02; visual box size=0.5 0.5 0.02
- added link box2_bottom_plate_back; collision box size=0.5 0.02 0.5; visual box size=0.5 0.02 0.5
- added link box2_bottom_plate_front; collision box size=0.5 0.02 0.5; visual box size=0.5 0.02 0.5
- added link box2_bottom_plate_left; collision box size=0.02 0.5 0.5; visual box size=0.02 0.5 0.5
- added link box2_bottom_plate_right; collision box size=0.02 0.5 0.5; visual box size=0.02 0.5 0.5
- added link box3_bottom_plate; collision box size=0.5 0.5 0.02; visual box size=0.5 0.5 0.02
- added link box3_bottom_plate_back; collision box size=0.5 0.02 0.5; visual box size=0.5 0.02 0.5
- added link box3_bottom_plate_front; collision box size=0.5 0.02 0.5; visual box size=0.5 0.02 0.5
- added link box3_bottom_plate_left; collision box size=0.02 0.5 0.5; visual box size=0.02 0.5 0.5
- added link box3_bottom_plate_right; collision box size=0.02 0.5 0.5; visual box size=0.02 0.5 0.5
- added link box4_bottom_plate; collision box size=0.5 0.5 0.02; visual box size=0.5 0.5 0.02
- added link box4_bottom_plate_back; collision box size=0.5 0.02 0.5; visual box size=0.5 0.02 0.5
- added link box4_bottom_plate_front; collision box size=0.5 0.02 0.5; visual box size=0.5 0.02 0.5
- added link box4_bottom_plate_left; collision box size=0.02 0.5 0.5; visual box size=0.02 0.5 0.5
- added link box4_bottom_plate_right; collision box size=0.02 0.5 0.5; visual box size=0.02 0.5 0.5
- added link box5_bottom_plate; collision box size=0.5 0.5 0.02; visual box size=0.5 0.5 0.02
- added link box5_bottom_plate_back; collision box size=0.5 0.02 0.5; visual box size=0.5 0.02 0.5
- added link box5_bottom_plate_front; collision box size=0.5 0.02 0.5; visual box size=0.5 0.02 0.5
- added link box5_bottom_plate_left; collision box size=0.02 0.5 0.5; visual box size=0.02 0.5 0.5
- added link box5_bottom_plate_right; collision box size=0.02 0.5 0.5; visual box size=0.02 0.5 0.5
Joints:
- removed joint base_link_to_crate0_joint
- removed joint base_link_to_crate1_joint
- removed joint base_link_to_crate2_joint
- removed joint base_link_to_crate_joint
- removed joint base_link_to_lamp0_joint
- removed joint base_link_to_lamp1_joint
- removed joint base_link_to_lamp2_joint
- added joint box1_bottom_plate_back_joint: type fixed, parent box1_bottom_plate, child box1_bottom_plate_back, origin xyz=0 -0.25 0.26 rpy=0 0 0
- added joint box1_bottom_plate_front_joint: type fixed, parent box1_bottom_plate, child box1_bottom_plate_front, origin xyz=0 0.25 0.26 rpy=0 0 0
- added joint box1_bottom_plate_joint: type fixed, parent base, child box1_bottom_plate, origin xyz=0 0 0 rpy=0 0 0
- added joint box1_bottom_plate_left_joint: type fixed, parent box1_bottom_plate, child box1_bottom_plate_left, origin xyz=-0.25 0 0.26 rpy=0 0 0
- added joint box1_bottom_plate_right_joint: type fixed, parent box1_bottom_plate, child box1_bottom_plate_right, origin xyz=0.25 0 0.26 rpy=0 0 0
- added joint box2_bottom_plate_back_joint: type fixed, parent box2_bottom_plate, child box2_bottom_plate_back, origin xyz=0 -0.25 0.26 rpy=0 0 0
- added joint box2_bottom_plate_front_joint: type fixed, parent box2_bottom_plate, child box2_bottom_plate_front, origin xyz=0 0.25 0.26 rpy=0 0 0
- added joint box2_bottom_plate_joint: type fixed, parent base, child box2_bottom_plate, origin xyz=0.5 0 0 rpy=0 0 0
- added joint box2_bottom_plate_left_joint: type fixed, parent box2_bottom_plate, child box2_bottom_plate_left, origin xyz=-0.25 0 0.26 rpy=0 0 0
- added joint box2_bottom_plate_right_joint: type fixed, parent box2_bottom_plate, child box2_bottom_plate_right, origin xyz=0.25 0 0.26 rpy=0 0 0
- added joint box3_bottom_plate_back_joint: type fixed, parent box3_bottom_plate, child box3_bottom_plate_back, origin xyz=0 -0.25 0.26 rpy=0 0 0
- added joint box3_bottom_plate_front_joint: type fixed, parent box3_bottom_plate, child box3_bottom_plate_front, origin xyz=0 0.25 0.26 rpy=0 0 0
- added joint box3_bottom_plate_joint: type fixed, parent base, child box3_bottom_plate, origin xyz=-0.5 0 0 rpy=0 0 0
- added joint box3_bottom_plate_left_joint: type fixed, parent box3_bottom_plate, child box3_bottom_plate_left, origin xyz=-0.25 0 0.26 rpy=0 0 0
- added joint box3_bottom_plate_right_joint: type fixed, parent box3_bottom_plate, child box3_bottom_plate_right, origin xyz=0.25 0 0.26 rpy=0 0 0
- added joint box4_bottom_plate_back_joint: type fixed, parent box4_bottom_plate, child box4_bottom_plate_back, origin xyz=0 -0.25 0.26 rpy=0 0 0
- added joint box4_bottom_plate_front_joint: type fixed, parent box4_bottom_plate, child box4_bottom_plate_front, origin xyz=0 0.25 0.26 rpy=0 0 0
- added joint box4_bottom_plate_joint: type fixed, parent base, child box4_bottom_plate, origin xyz=0 0.5 0 rpy=0 0 0
- added joint box4_bottom_plate_left_joint: type fixed, parent box4_bottom_plate, child box4_bottom_plate_left, origin xyz=-0.25 0 0.26 rpy=0 0 0
- added joint box4_bottom_plate_right_joint: type fixed, parent box4_bottom_plate, child box4_bottom_plate_right, origin xyz=0.25 0 0.26 rpy=0 0 0
- added joint box5_bottom_plate_back_joint: type fixed, parent box5_bottom_plate, child box5_bottom_plate_back, origin xyz=0 -0.25 0.26 rpy=0 0 0
- added joint box5_bottom_plate_front_joint: type fixed, parent box5_bottom_plate, child box5_bottom_plate_front, origin xyz=0 0.25 0.26 rpy=0 0 0
- added joint box5_bottom_plate_joint: type fixed, parent base, child box5_bottom_plate, origin xyz=0 -0.5 0 rpy=0 0 0
- added joint box5_bottom_plate_left_joint: type fixed, parent box5_bottom_plate, child box5_bottom_plate_left, origin xyz=-0.25 0 0.26 rpy=0 0 0
- added joint box5_bottom_plate_right_joint: type fixed, parent box5_bottom_plate, child box5_bottom_plate_right, origin xyz=0.25 0 0.26 rpy=0 0 0

File: panda_four_description/urdf/panda_four_binpick.urdf.xacro (robot description, xacro)
@@ -7,4 +7,5 @@
   <xacro:include filename="$(find moveit_resources_panda_description)/urdf/panda_arm.xacro"/>
   <xacro:include filename="$(find moveit_resources_panda_description)/urdf/hand.xacro"/>
+  <xacro:include filename="box.xacro"/>
   <!-- box shaped table as base for the 4 Pandas -->
   <link name="base">
@@ -25,137 +26,14 @@
     </collision>
   </link>
-  <joint name="base_link_to_crate0_joint" type="fixed">
-    <parent link="base"/>
-    <child link="crate0"/>
-    <origin xyz="0.53 0.1 0.1" rpy="0 0 1.57"/>
-  </joint>
-  <link name="crate0">
-    <visual>
-      <origin rpy="0 0 0" xyz="0.0 0.0 0.0"/>
-      <geometry>
-        <mesh filename="/root/catkin_ws/src/moveit_configs/stl/crate.stl" scale="0.01 0.01 0.01"/>
-      </geometry>
-    </visual>
-    <collision>
-      <origin rpy="0 0 0" xyz="0.0 0.0 0.0"/>
-      <geometry>
-        <mesh filename="/root/catkin_ws/src/moveit_configs/stl/crate.stl" scale="0.01 0.01 0.01"/>
-      </geometry>
-    </collision>
-  </link>
-  <joint name="base_link_to_crate_joint" type="fixed">
-    <parent link="base"/>
-    <child link="crate"/>
-    <origin xyz="0.13 0.1 0.1" rpy="0 0 1.57"/>
-  </joint>
-  <link name="crate">
-    <visual>
-      <origin rpy="0 0 0" xyz="0.0 0.0 0.0"/>
-      <geometry>
-        <mesh filename="/root/catkin_ws/src/moveit_configs/stl/crate.stl" scale="0.01 0.01 0.01"/>
-      </geometry>
-    </visual>
-    <collision>
-      <origin rpy="0 0 0" xyz="0.0 0.0 0.0"/>
-      <geometry>
-        <mesh filename="/root/catkin_ws/src/moveit_configs/stl/crate.stl" scale="0.01 0.01 0.01"/>
-      </geometry>
-    </collision>
-  </link>
-  <joint name="base_link_to_crate1_joint" type="fixed">
-    <parent link="base"/>
-    <child link="crate1"/>
-    <origin xyz="-0.27 0.1 0.1" rpy="0 0 1.57"/>
-  </joint>
-  <link name="crate1">
-    <visual>
-      <origin rpy="0 0 0" xyz="0.0 0.0 0.0"/>
-      <geometry>
-        <mesh filename="/root/catkin_ws/src/moveit_configs/stl/crate.stl" scale="0.01 0.01 0.01"/>
-      </geometry>
-    </visual>
-    <collision>
-      <origin rpy="0 0 0" xyz="0.0 0.0 0.0"/>
-      <geometry>
-        <mesh filename="/root/catkin_ws/src/moveit_configs/stl/crate.stl" scale="0.01 0.01 0.01"/>
-      </geometry>
-    </collision>
-  </link>
-  <joint name="base_link_to_crate2_joint" type="fixed">
-    <parent link="base"/>
-    <child link="crate2"/>
-    <origin xyz="-0.67 0.1 0.1" rpy="0 0 1.57"/>
-  </joint>
-  <link name="crate2">
-    <visual>
-      <origin rpy="0 0 0" xyz="0.0 0.0 0.0"/>
-      <geometry>
-        <mesh filename="/root/catkin_ws/src/moveit_configs/stl/crate.stl" scale="0.01 0.01 0.01"/>
-      </geometry>
-    </visual>
-    <collision>
-      <origin rpy="0 0 0" xyz="0.0 0.0 0.0"/>
-      <geometry>
-        <mesh filename="/root/catkin_ws/src/moveit_configs/stl/crate.stl" scale="0.01 0.01 0.01"/>
-      </geometry>
-    </collision>
-  </link>
-  <joint name="base_link_to_lamp0_joint" type="fixed">
-    <parent link="base"/>
-    <child link="lamp0"/>
-    <origin xyz="0.5 0.0 0.8" rpy="0 0 0"/>
-  </joint>
-  <link name="lamp0">
-    <visual>
-      <origin rpy="0 0 0" xyz="0.0 0.0 0.0"/>
-      <geometry>
-        <mesh filename="/root/catkin_ws/src/moveit_configs/stl/lamp.stl" scale="0.000027 0.000027 0.000027"/>
-      </geometry>
-    </visual>
-    <collision>
-      <origin rpy="0 0 0" xyz="0.0 0.0 0.0"/>
-      <geometry>
-        <mesh filename="/root/catkin_ws/src/moveit_configs/stl/crate.stl" scale="0.01 0.01 0.01"/>
-      </geometry>
-    </collision>
-  </link>
-  <joint name="base_link_to_lamp1_joint" type="fixed">
-    <parent link="base"/>
-    <child link="lamp1"/>
-    <origin xyz="0.0 0.0 1.13" rpy="0 0 0"/>
-  </joint>
-  <link name="lamp1">
-    <visual>
-      <origin rpy="0 0 0" xyz="0.0 0.0 0.0"/>
-      <geometry>
-        <mesh filename="/root/catkin_ws/src/moveit_configs/stl/lamp.stl" scale="0.000027 0.000032 0.000032"/>
-      </geometry>
-    </visual>
-    <collision>
-      <origin rpy="0 0 0" xyz="0.0 0.0 0.0"/>
-      <geometry>
-        <mesh filename="/root/catkin_ws/src/moveit_configs/stl/crate.stl" scale="0.01 0.01 0.01"/>
-      </geometry>
-    </collision>
-  </link>
-  <joint name="base_link_to_lamp2_joint" type="fixed">
-    <parent link="base"/>
-    <child link="lamp2"/>
-    <origin xyz="-0.5 0.0 0.8" rpy="0 0 0"/>
-  </joint>
-  <link name="lamp2">
-    <visual>
-      <origin rpy="0 0 0" xyz="0.0 0.0 0.0"/>
-      <geometry>
-        <mesh filename="/root/catkin_ws/src/moveit_configs/stl/lamp.stl" scale="0.000027 0.000027 0.000027"/>
-      </geometry>
-    </visual>
-    <collision>
-      <origin rpy="0 0 0" xyz="0.0 0.0 0.0"/>
-      <geometry>
-        <mesh filename="/root/catkin_ws/src/moveit_configs/stl/crate.stl" scale="0.01 0.01 0.01"/>
-      </geometry>
-    </collision>
-  </link>
+  <xacro:add_box parent_link="base" box_name="box1" box_length="0.5" box_width="0.5"
+      box_height="0.5" box_x="0" box_y="0" box_z="0" box_color="0 0 1 1"/>
+  <xacro:add_box parent_link="base" box_name="box2" box_length="0.5" box_width="0.5"
+      box_height="0.5" box_x="0.5" box_y="0" box_z="0" box_color="0 1 0 1"/>
+  <xacro:add_box parent_link="base" box_name="box3" box_length="0.5" box_width="0.5"
+     box_height="0.5" box_x="-0.5" box_y="0" box_z="0" box_color="1 0 0 1"/>
+  <xacro:add_box parent_link="base" box_name="box4" box_length="0.5" box_width="0.5"
+     box_height="0.5" box_x="0" box_y="0.5" box_z="0" box_color="1 1 0 1"/>
+  <xacro:add_box parent_link="base" box_name="box5" box_length="0.5" box_width="0.5"
+     box_height="0.5" box_x="0" box_y="-0.5" box_z="0" box_color="0.5 0 0.5 1"/>
   <!-- panda_0 with gripper -->
   <xacro:panda_arm arm_id="$(arg arm_id_0)" connected_to="base"  xyz="0.4 -0.4 0.1" rpy="0 0 2.28"/>

Commit message: adding rods for four_bins scene and 10 poses

File: panda_four_description/urdf/panda_four_binpick.urdf (robot description, URDF)
Before this commit: robot panda, 74 links, 73 joints
Links:
- added link rod_0; collision rod length=0.5 radius=0.015; visual rod length=0.5 radius=0.015
- added link rod_1; collision rod length=0.5 radius=0.015; visual rod length=0.5 radius=0.015
- added link rod_2; collision rod length=0.5 radius=0.015; visual rod length=0.5 radius=0.015
- added link rod_3; collision rod length=0.5 radius=0.015; visual rod length=0.5 radius=0.015
Joints:
- added joint rod_0_joint: type fixed, parent panda0_hand, child rod_0, origin xyz=0 0 0.1 rpy=0 1.5708 0
- added joint rod_1_joint: type fixed, parent panda1_hand, child rod_1, origin xyz=0 0 0.1 rpy=0 1.5708 0
- added joint rod_2_joint: type fixed, parent panda0_hand, child rod_2, origin xyz=0 0 0.1 rpy=0 1.5708 0
- added joint rod_3_joint: type fixed, parent panda0_hand, child rod_3, origin xyz=0 0 0.1 rpy=0 1.5708 0

File: panda_two_description/urdf/panda_two_objects.urdf.xacro (robot description, xacro)
@@ -52,8 +52,8 @@
   <xacro:panda_arm arm_id="$(arg arm_id_0)" connected_to="base"  xyz="0.4 0.0 0.1" rpy="0 0 -3.141592653589793"/>
   <xacro:hand ns="$(arg arm_id_0)" rpy="0 0 0" connected_to="$(arg arm_id_0)_link8"/>
-  <xacro:add_rod parent_link="$(arg arm_id_0)_hand" rod_name="rod_0" rod_length="0.5" rod_radius="0.015" rod_color="0.5 0.5 0.5 1"/>
+  <xacro:add_rod parent_link="$(arg arm_id_0)_hand" rod_name="rod_0" rod_length="0.5" rod_radius="0.015" rod_color="0 1 0 1"/>
   <!-- panda_1 with gripper -->
   <xacro:panda_arm arm_id="$(arg arm_id_1)" connected_to="base"  xyz="-0.4 0.0 0.1" rpy="0 0 0"/>
   <xacro:hand ns="$(arg arm_id_1)" rpy="0 0 0" connected_to="$(arg arm_id_1)_link8"/>
-  <xacro:add_rod parent_link="$(arg arm_id_1)_hand" rod_name="rod_1" rod_length="0.5" rod_radius="0.015" rod_color="0.5 0.5 0.5 1"/>
+  <xacro:add_rod parent_link="$(arg arm_id_1)_hand" rod_name="rod_1" rod_length="0.5" rod_radius="0.015" rod_color="0 0 1 1"/>
 </robot>
