Commit message: add a new three panda arm configuration around a table

File: panda_three_description/urdf/panda_three_round.urdf (robot description, URDF)
Before this commit: robot panda, 46 links, 45 joints
Links:
- removed link back_plate
- removed link left_side_plate
- removed link right_side_plate
- removed link shelf0
- removed link shelf1
- removed link shelf2
- removed link shelf3
- removed link shelf4
- removed link wall
Joints:
- removed joint back_plate_joint
- removed joint left_side_plate_joint
- removed joint right_side_plate_joint
- removed joint shelf0_joint
- removed joint shelf1_joint
- removed joint shelf2_joint
- removed joint shelf3_joint
- removed joint shelf4_joint
- removed joint wall_joint
- joint panda0_joint_base: origin xyz=-0.4 0 0.1 rpy=0 0 1.5708 -> xyz=1.21 0 0 rpy=0 0 3.1415927
- joint panda1_joint_base: origin xyz=0 0.0 0.1 rpy=0 0 1.5708 -> xyz=0.22 0.571577 0 rpy=0 0 -1.04741975
- joint panda2_joint_base: origin xyz=0.4 0 0.1 rpy=0 0 1.5708 -> xyz=0.22 -0.571577 0 rpy=0 0 1.04741975
