Commit message: update dual_gp4 moveit config

File: dual_gp4_moveit_config/config/gazebo_dual_gp4.urdf (robot description, URDF)
Before this commit: robot dual_gp4, 30 links, 29 joints
Joints:
- joint left_arm_to_base: origin xyz=0 0 0 rpy=0 0 0 -> xyz=0 0 0.9246 rpy=0 0 0
- joint right_arm_to_base: origin xyz=0.7951 0 0 rpy=0 0 3.141592653589793 -> xyz=0.7951 0 0.9246 rpy=0 0 3.141592653589793

Commit message: update dual arm srdf

File: dual_gp4_moveit_config/config/gazebo_dual_gp4.urdf (robot description, URDF)
Before this commit: robot dual_gp4, 30 links, 29 joints
Links:
- added link left_arm_link_mountplate, mass 0.10811; collision mesh filename=file:///home/philip/catkin_ws/src/robot_digital_twin/meshes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; visual mesh filename=file:///home/philip/catkin_ws/src/robot_digital_twin/meshes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
- added link right_arm_link_mountplate, mass 0.10811; collision mesh filename=file:///home/philip/catkin_ws/src/robot_digital_twin/meshes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; visual mesh filename=file:///home/philip/catkin_ws/src/robot_digital_twin/meshes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
- link left_arm_base_link: geometry collision mesh filename=file:///home/philip/catkin_ws/src/robot_digital_twin/meshes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; visual mesh filename=file:///home/philip/catkin_ws/src/robot_digital_twin/meshes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
- link left_arm_fts: geometry collision cylinder length=0.0505 radius=0.058; visual cylinder length=0.0505 radius=0.0472
- link left_arm_link_1: geometry collision mesh filename=file:///home/philip/catkin_ws/src/robot_digital_twin/meshes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; visual mesh filename=file:///home/philip/catkin_ws/src/robot_digital_twin/meshes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
- link left_arm_link_2: geometry collision mesh filename=file:///home/philip/catkin_ws/src/robot_digital_twin/meshes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; visual mesh filename=file:///home/philip/catkin_ws/src/robot_digital_twin/meshes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
- link left_arm_link_3: geometry collision mesh filename=file:///home/philip/catkin_ws/src/robot_digital_twin/meshes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; visual mesh filename=file:///home/philip/catkin_ws/src/robot_digital_twin/meshes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
- link left_arm_link_4: geometry collision mesh filename=file:///home/philip/catkin_ws/src/robot_digital_twin/meshes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; visual mesh filename=file:///home/philip/catkin_ws/src/robot_digital_twin/meshes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
- link left_arm_link_5: geometry collision mesh filename=file:///home/philip/catkin_ws/src/robot_digital_twin/meshes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; visual mesh filename=file:///home/philip/catkin_ws/src/robot_digital_twin/meshes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
- link left_arm_link_6: geometry collision mesh filename=file:///home/philip/catkin_ws/src/robot_digital_twin/meshes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; visual mesh filename=file:///home/philip/catkin_ws/src/robot_digital_twin/meshes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
- link left_arm_link_camera: geometry collision mesh filename=file:///home/philip/catkin_ws/src/robot_digital_twin/meshes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; visual mesh filename=file:///home/philip/catkin_ws/src/robot_digital_twin/meshes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
- link left_arm_link_camera_origin: geometry visual box size=0.0001 0.002 0.001
- link left_arm_link_tool: geometry collision mesh filename=file:///home/philip/catkin_ws/src/robot_digital_twin/meshes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; visual mesh filename=file:///home/philip/catkin_ws/src/robot_digital_twin/meshes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
- link right_arm_base_link: geometry collision mesh filename=file:///home/philip/catkin_ws/src/robot_digital_twin/meshes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; visual mesh filename=file:///home/philip/catkin_ws/src/robot_digital_twin/meshes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
- link right_arm_fts: geometry collision cylinder length=0.0505 radius=0.058; visual cylinder length=0.0505 radius=0.0472
- link right_arm_link_1: geometry collision mesh filename=file:///home/philip/catkin_ws/src/robot_digital_twin/meshes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; visual mesh filename=file:///home/philip/catkin_ws/src/robot_digital_twin/meshes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
- link right_arm_link_2: geometry collision mesh filename=file:///home/philip/catkin_ws/src/robot_digital_twin/meshes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; visual mesh filename=file:///home/philip/catkin_ws/src/robot_digital_twin/meshes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
- link right_arm_link_3: geometry collision mesh filename=file:///home/philip/catkin_ws/src/robot_digital_twin/meshes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; visual mesh filename=file:///home/philip/catkin_ws/src/robot_digital_twin/meshes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
- link right_arm_link_4: geometry collision mesh filename=file:///home/philip/catkin_ws/src/robot_digital_twin/meshes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; visual mesh filename=file:///home/philip/catkin_ws/src/robot_digital_twin/meshes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
- link right_arm_link_5: geometry collision mesh filename=file:///home/philip/catkin_ws/src/robot_digital_twin/meshes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; visual mesh filename=file:///home/philip/catkin_ws/src/robot_digital_twin/meshes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
- link right_arm_link_6: geometry collision mesh filename=file:///home/philip/catkin_ws/src/robot_digital_twin/meshes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; visual mesh filename=file:///home/philip/catkin_ws/src/robot_digital_twin/meshes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
- link right_arm_link_camera: geometry collision mesh filename=file:///home/philip/catkin_ws/src/robot_digital_twin/meshes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; visual mesh filename=file:///home/philip/catkin_ws/src/robot_digital_twin/meshes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
- link right_arm_link_camera_origin: geometry visual box size=0.0001 0.002 0.001
- link right_arm_link_tool: geometry collision mesh filename=file:///home/philip/catkin_ws/src/robot_digital_twin/meshes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; visual mesh filename=file:///home/philip/catkin_ws/src/robot_digital_twin/meshes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
Joints:
- removed joint left_arm_tool_precam
- removed joint right_arm_tool_precam
- added joint left_arm_fts_plate: type fixed, parent left_arm_fts, child left_arm_link_mountplate, origin xyz=0 0 0.02526 rpy=1.5707963267948966 0 0
- added joint left_arm_plate_precam: type fixed, parent left_arm_link_mountplate, child left_arm_link_precam, origin xyz=0 0 0 rpy=-1.5707963267948966 0  0
- added joint right_arm_fts_plate: type fixed, parent right_arm_fts, child right_arm_link_mountplate, origin xyz=0 0 0.02526 rpy=1.5707963267948966 0 0
- added joint right_arm_plate_precam: type fixed, parent right_arm_link_mountplate, child right_arm_link_precam, origin xyz=0 0 0 rpy=-1.5707963267948966 0  0
- joint left_arm_camera_imgplane: origin xyz=0.013 0.0 0.0305 rpy=0 0 0 -> xyz=0.009 0 0 rpy=0 4.71238898038469 -1.5707963267948966
- joint left_arm_fts_tool: origin xyz=0 0 0.02525 rpy=0 0 3.141592653589793 -> xyz=0 0 0.027790000000000002 rpy=0 0 3.141592653589793
- joint left_arm_precam_camera: origin xyz=0 0 0 rpy=0 0.7853981633974483 0 -> xyz=0 0.053512 0.02555 rpy=0  0  0
- joint right_arm_camera_imgplane: origin xyz=0.013 0.0 0.0305 rpy=0 0 0 -> xyz=0.009 0 0 rpy=0 4.71238898038469 -1.5707963267948966
- joint right_arm_fts_tool: origin xyz=0 0 0.02525 rpy=0 0 3.141592653589793 -> xyz=0 0 0.027790000000000002 rpy=0 0 3.141592653589793
- joint right_arm_precam_camera: origin xyz=0 0 0 rpy=0 0.7853981633974483 0 -> xyz=0 0.053512 0.02555 rpy=0  0  0
- joint right_arm_to_base: origin xyz=0.7951 0 0.9246 rpy=0 0 3.141592653589793 -> xyz=0.88047659 -0.01305078 0.9246 rpy=0 0 3.13422265
